File: ecad/_autosave-Iridium-adc.kicad_pcb (KiCad board)
At the start: 2 copper layers, 82.5 x 70 mm, 122 parts, among them J1 +15V, J2 XLR3, J4 Nucleo_F446_LHS, J5 Nucleo_F446_RHS, U1 ADR434BRZ, U10 NCV1117ST25T3G, U11 CB3-3C-40M0000, U12 NC7SZ08M5, U13 AD7760, U2 OPA207IDR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

Commit message: Mostly complete schematic, about to tape out the PCB.
Parts:
- moved U13 280.4 mm to (-76.8, 108.8)
Changed lines of the file:
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@@
     (links 282)
     (no_connects 91)
-    (area 16.924999 36.424999 99.575001 106.575001)
+    (area -98.525 60.49857 209.875001 135.136667)
     (thickness 1.6)
     (drawings 4)
@@
   )
   (module Housings_QFP:LQFP-64_10x10mm_Pitch0.5mm (layer F.Cu)
-    (at 203.2 94.6 180)
+    (at -76.8 108.8 180)
     (descr "64 LEAD LQFP 10x10mm (see MICREL LQFP10x10-64LD-PL-1.pdf)")
     (tags "QFP 0.5")
