File: ecad/Iridium-adc.kicad_pcb (KiCad board)
At the start: 2 copper layers, 82.5 x 70 mm, 122 parts, among them J1 +15V, J2 XLR3, J4 Nucleo_F446_LHS, J5 Nucleo_F446_RHS, U1 ADR434BRZ, U10 NCV1117ST25T3G, U11 CB3-3C-40M0000, U12 NC7SZ08M5, U13 AD7760, U2 OPA207IDR, U3 ADP7104ARDZ-R7, U4 OPA207IDR, U5 ADP7104ARDZ-5.0-R7, U6 OPA1612, U7 OPA1632, U8 OPA1632, U9 OPA1632

Commit message: First complete pass of PCB with preamp, ADC, and nucleo dev board connections.
Parts:
- removed C32: 120p, Capacitors_SMD:C_0603_HandSoldering
- removed C33, C8: 0.1u, Capacitors_SMD:C_0603_HandSoldering
- removed C34, C35: 10p, Capacitors_SMD:C_0603_HandSoldering
- removed C36: 1n, Capacitors_SMD:C_0603_HandSoldering
- removed R5, R6: 10k, Resistors_SMD:R_0603_HandSoldering
- removed REF**: Billtech_back, feetprints:Billtech_back
- removed U4: OPA207IDR, Housings_SOIC:SOIC-8_3.9x4.9mm_Pitch1.27mm
- removed U9: OPA1632, Housings_SOIC:SOIC-8_3.9x4.9mm_Pitch1.27mm
- C30: value 0.1u -> 120p
- C31, R31, R33: moved to B.Cu
- C42, C53, C54, C56: footprint Capacitors_SMD:C_0603_HandSoldering -> Capacitors_SMD:C_0603; moved to B.Cu
- C43: value 100n -> 0.1u; footprint Capacitors_SMD:C_0603_HandSoldering -> Capacitors_SMD:C_0603
- C44, C45, C46, C47, C48, C50, C51, C52, C55: value 100n -> 0.1u; footprint Capacitors_SMD:C_0603_HandSoldering -> Capacitors_SMD:C_0603; moved to B.Cu
- C49: footprint Capacitors_SMD:C_0603_HandSoldering -> Capacitors_SMD:C_0603
- C7: value 22u -> 0.1u; footprint Capacitors_SMD:C_1210_HandSoldering -> Capacitors_SMD:C_0603_HandSoldering; moved to B.Cu
- L10: footprint Inductors_SMD:L_0603_HandSoldering -> Inductors_SMD:L_0603
- R34, R35, R36: footprint Inductors_SMD:L_0603_HandSoldering -> Resistors_SMD:R_0603
- U13: footprint Housings_QFP:LQFP-64_10x10mm_Pitch0.5mm -> feetprints:LQFP-EP-64_10x10mm_Pitch0.5mm_6mm_square_paddle
- moved J4 209.5 mm to (151.2, 126.1), turned to 90 degrees
- moved J5 209.1 mm to (150.7, 65.1), turned to 90 degrees
- moved L6 136.8 mm to (190.3, 80.7), turned to 180 degrees
- moved L11 136.3 mm to (190.5, 83.6), turned to 270 degrees
- moved C52 133.9 mm to (188.7, 86.5), turned to 180 degrees
- moved L1 133.7 mm to (186.8, 79.5), turned to 180 degrees
- moved C48 130.6 mm to (185.0, 85.0), turned to 270 degrees
- moved R35 130.6 mm to (183.8, 80.7), turned to 90 degrees
- moved C43 130.6 mm to (184.3, 82.7), turned to 180 degrees
- moved L7 129.8 mm to (182.3, 78.5), turned to 270 degrees
- moved C55 129.1 mm to (183.4, 85.0), turned to 270 degrees
- moved C49 128.8 mm to (182.3, 82.0), turned to 270 degrees
- moved L9 128.2 mm to (180.7, 78.5), turned to 270 degrees
- moved C50 128.2 mm to (184.7, 95.5), turned to 90 degrees
- moved L8 127.9 mm to (184.9, 99.0), turned to 90 degrees
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Connections:
- net /Microcontroller/DB8 renamed Net-(J4-Pad9)
- C26 pad 1: Net-(C26-Pad1) -> /ADC/InputP
- C27 pad 1: Net-(C27-Pad1) -> /ADC/InputN
- C29 pad 1: Net-(C29-Pad1) -> /ADC/VINAN
- C29 pad 2: Net-(C29-Pad2) -> /ADC/VINAP
- C30 pad 1: /Input/OCM -> /ADC/VOUTAN
- C30 pad 2: GND -> /ADC/VINAP
- C31 pad 1: Net-(C31-Pad1) -> /ADC/VOUTAP
- C31 pad 2: Net-(C29-Pad1) -> /ADC/VINAN
- C7 pad 1: Net-(C7-Pad1) -> /Input/BIAS
- J4 pad 1: /Microcontroller/DB10 -> /ADC/~SYNC
- J4 pad 10: GND -> Net-(J4-Pad10)
- J4 pad 11: /Microcontroller/PB7 -> Net-(J4-Pad11)
- J4 pad 12: /Microcontroller/DB13 -> /Microcontroller/IOREF
- J4 pad 13: /Microcontroller/DB14 -> /ADC/~RD
- J4 pad 14: /Microcontroller/DB15 -> /Microcontroller/RESET
- J4 pad 15: /Microcontroller/PH0 -> /ADC/~CS
- J4 pad 16: /Microcontroller/PH1 -> /Microcontroller/3V3
- J4 pad 17: /Microcontroller/VBAT -> /ADC/DB15
- J4 pad 18: /Microcontroller/PC2 -> /Microcontroller/5V
- J4 pad 19: /Microcontroller/PC3 -> GND
- J4 pad 2: /Microcontroller/DB12 -> /ADC/~RESET
- J4 pad 20: /Microcontroller/PC0 -> GND
- J4 pad 21: /Microcontroller/DB9 -> /Microcontroller/PB7
- J4 pad 22: /Microcontroller/PB0 -> GND
- J4 pad 23: /Microcontroller/DB2 -> /ADC/DB14
- J4 pad 24: /Microcontroller/DB1 -> /Microcontroller/Vin
- J4 pad 25: /Microcontroller/DB0 -> /ADC/DB13
- J4 pad 27: /Microcontroller/Vin -> /ADC/DB12
- J4 pad 28: GND -> /ADC/DB11
- J4 pad 29: GND -> /Microcontroller/PH0
- J4 pad 3: /Microcontroller/VDD -> /ADC/~DRDY
- J4 pad 30: /Microcontroller/5V -> /ADC/DB10
- J4 pad 31: /Microcontroller/3V3 -> /Microcontroller/PH1
- J4 pad 32: /Microcontroller/RESET -> /ADC/DB9
- J4 pad 33: /Microcontroller/IOREF -> /Microcontroller/VBAT
- J4 pad 34: Net-(J4-Pad34) -> /Microcontroller/PB0
- J4 pad 35: GND -> /Microcontroller/PC2
- J4 pad 36: /Microcontroller/E5V -> /ADC/DB8
- J4 pad 37: /Microcontroller/PD2 -> /Microcontroller/PC3
- J4 pad 38: /Microcontroller/DB11 -> /Microcontroller/PC0
- J4 pad 4: /Microcontroller/BOOT0 -> /Microcontroller/PD2
- J4 pad 5: Net-(J4-Pad5) -> /Microcontroller/VDD
- J4 pad 6: Net-(J4-Pad6) -> /Microcontroller/E5V
- J4 pad 7: /Microcontroller/DB6 -> /Microcontroller/BOOT0
- J4 pad 8: /Microcontroller/DB7 -> GND
- J5 pad 10: /Microcontroller/PC7 -> Net-(J5-Pad10)
- J5 pad 11: /Microcontroller/DB4 -> /Microcontroller/PA5
- J5 pad 12: /Microcontroller/DB3 -> /ADC/DB3
- J5 pad 13: /Microcontroller/PB10 -> /Microcontroller/PA6
- J5 pad 14: /Microcontroller/PB4 -> /ADC/DB4
- J5 pad 15: /Microcontroller/PB5 -> /Microcontroller/PA7
- J5 pad 16: /Microcontroller/PB3 -> /Microcontroller/PB12
- J5 pad 17: /Microcontroller/DB5 -> /Microcontroller/PB6
- J5 pad 18: /Microcontroller/PA2 -> Net-(J5-Pad18)
- J5 pad 19: /Microcontroller/PA3 -> /Microcontroller/PC7
- J5 pad 2: /Microcontroller/PB8 -> /ADC/DB0
- J5 pad 20: Net-(J5-Pad20) -> GND
- J5 pad 21: Net-(J5-Pad21) -> /ADC/DB5
- J5 pad 22: /Microcontroller/PC4 -> /Microcontroller/PB2
- J5 pad 23: GND -> /ADC/DB6
- J5 pad 24: /Microcontroller/PB13 -> /Microcontroller/PB1
- J5 pad 25: /Microcontroller/PB14 -> /Microcontroller/PB10
- J5 pad 27: /Microcontroller/PB1 -> /Microcontroller/PB4
- J5 pad 28: /Microcontroller/PB2 -> /Microcontroller/PB14
- J5 pad 29: GND -> /Microcontroller/PB5
- J5 pad 3: /Microcontroller/PB9 -> /Microcontroller/PB8
- J5 pad 30: Net-(J5-Pad30) -> /Microcontroller/PB13
- J5 pad 31: /Microcontroller/PB12 -> /Microcontroller/PB3
- J5 pad 32: /ADC/~RD -> GND
- J5 pad 33: /ADC/~SYNC -> /ADC/DB7
- J5 pad 34: Net-(J5-Pad34) -> /Microcontroller/PC4
- J5 pad 35: /Microcontroller/U5V -> /Microcontroller/PA2
- J5 pad 36: /ADC/~DRDY -> Net-(J5-Pad36)
- J5 pad 37: /ADC/~RESET -> /Microcontroller/PA3
- J5 pad 38: /ADC/~CS -> Net-(J5-Pad38)
- J5 pad 4: /Microcontroller/AVDD -> /ADC/DB1
- J5 pad 5: GND -> /Microcontroller/PB9
- J5 pad 6: /Microcontroller/PA5 -> /ADC/DB2
- J5 pad 7: /Microcontroller/PA6 -> /Microcontroller/AVDD
- J5 pad 8: /Microcontroller/PA7 -> /Microcontroller/U5V
- J5 pad 9: /Microcontroller/PB6 -> GND
- R26 pad 1: Net-(C26-Pad1) -> /ADC/InputP
- R27 pad 1: Net-(C27-Pad1) -> /ADC/InputN
- R28 pad 1: Net-(C29-Pad1) -> /ADC/VINAP
- R28 pad 2: Net-(C26-Pad1) -> /ADC/InputP
- R29 pad 1: Net-(C29-Pad2) -> /ADC/VINAN
- R29 pad 2: Net-(C27-Pad1) -> /ADC/InputN
- R30 pad 1: Net-(C31-Pad1) -> /ADC/VOUTAN
- R30 pad 2: Net-(C29-Pad1) -> /ADC/VINAP
- R31 pad 1: Net-(C32-Pad1) -> /ADC/VOUTAP
- R31 pad 2: Net-(C29-Pad2) -> /ADC/VINAN
- R32 pad 1: /ADC/InputP -> /ADC/VINP
- R32 pad 2: Net-(C31-Pad1) -> /ADC/VOUTAP
- R33 pad 1: /ADC/InputN -> /ADC/VINN
- R33 pad 2: Net-(C32-Pad1) -> /ADC/VOUTAN
- U13 pad 19: Net-(U13-Pad19) -> /ADC/VINAP
- U13 pad 20: Net-(U13-Pad20) -> /ADC/VINAN
- U13 pad 21: Net-(U13-Pad21) -> /ADC/VOUTAN
- U13 pad 22: Net-(U13-Pad22) -> /ADC/VOUTAP
- U13 pad 25: /ADC/InputP -> /ADC/VINP
- U13 pad 26: /ADC/InputN -> /ADC/VINN
- U13 pad 57: /ADC/DB3 -> /ADC/DB4
- U13 pad 58: /ADC/DB4 -> /ADC/DB3
- U13 pad 60: /ADC/DB0 -> /ADC/DB1
- U13 pad 61: /ADC/DB1 -> /ADC/DB0
- U8 pad 4: Net-(C27-Pad1) -> /ADC/InputN
- U8 pad 5: Net-(C26-Pad1) -> /ADC/InputP
Routing:
- net +5V: track 8.40 -> 88.1 mm, vias 0 -> 4
- net +12V: track 219.2 -> 140.9 mm, vias 8 -> 2
- net GND: track 187.1 -> 262.1 mm, vias 38 -> 63
- net /ADC/~SYNC: track 0.00 -> 63.2 mm
- net /ADC/DB0: track 0.00 -> 59.2 mm
- net /ADC/~DRDY: track 0.00 -> 58.7 mm
- net /ADC/~RESET: track 0.00 -> 58.5 mm
- net /ADC/DB1: track 0.00 -> 57.7 mm
- net /ADC/DB2: track 0.00 -> 56.2 mm
- net +2V5: track 0.00 -> 53.1 mm, vias 0 -> 2
- net /ADC/DB3: track 0.00 -> 49.8 mm
- net /ADC/DB4: track 0.00 -> 48.3 mm
- net /ADC/~RD: track 0.00 -> 46.3 mm
- net /ADC/~CS: track 0.00 -> 44.4 mm
- net /ADC/DB15: track 0.00 -> 40.7 mm
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- added copper zone on B.Cu, net GND
Other:
- rule trace_min: 0.2 -> 0.1524
- rule via_min_drill: 0.3 -> 0.254
- board text added: "+ -"

Commit message: Rev A of board as ordered from Osh Park.
Parts:
- added G***: LOGO, feetprints:IridiumADC, F.Cu at (134.6, 121.9)
- added REF**: Billtech, feetprints:Billtech, F.Cu at (135.9, 64.8)
- C7: moved to F.Cu
- J2: footprint Pin_Headers:Pin_Header_Straight_1x03_Pitch2.54mm -> Pin_Headers:Pin_Header_Straight_1x04_Pitch2.54mm
- R11: value 1MR -> 1M
- U3: value ADP7104ARDZ-R7 -> ADP7105ARDZ
- U5: value ADP7104ARDZ-5.0-R7 -> ADP7104ARDZ-5.0
- moved C7 37.2 mm to (124.7, 86.0)
- moved C17 2.10 mm to (139.0, 85.2)
- moved C18 2.10 mm to (139.0, 89.2)
- moved C37 1.90 mm to (141.0, 85.2)
- moved C38 1.90 mm to (141.0, 89.2)
Connections:
- J4 pad 10: Net-(J4-Pad10) -> (no net)
- J4 pad 11: Net-(J4-Pad11) -> (no net)
- J4 pad 12: /Microcontroller/IOREF -> (no net)
- J4 pad 14: /Microcontroller/RESET -> (no net)
- J4 pad 16: /Microcontroller/3V3 -> (no net)
- J4 pad 18: /Microcontroller/5V -> (no net)
- J4 pad 21: /Microcontroller/PB7 -> (no net)
- J4 pad 24: /Microcontroller/Vin -> (no net)
- J4 pad 26: Net-(J4-Pad26) -> (no net)
- J4 pad 29: /Microcontroller/PH0 -> (no net)
- J4 pad 31: /Microcontroller/PH1 -> (no net)
- J4 pad 33: /Microcontroller/VBAT -> (no net)
- J4 pad 34: /Microcontroller/PB0 -> (no net)
- J4 pad 35: /Microcontroller/PC2 -> (no net)
- J4 pad 37: /Microcontroller/PC3 -> (no net)
- J4 pad 38: /Microcontroller/PC0 -> (no net)
- J4 pad 4: /Microcontroller/PD2 -> (no net)
- J4 pad 5: /Microcontroller/VDD -> (no net)
- J4 pad 6: /Microcontroller/E5V -> (no net)
- J4 pad 7: /Microcontroller/BOOT0 -> (no net)
- J4 pad 9: Net-(J4-Pad9) -> (no net)
- J5 pad 1: /Microcontroller/PC9 -> (no net)
- J5 pad 10: Net-(J5-Pad10) -> (no net)
- J5 pad 11: /Microcontroller/PA5 -> (no net)
- J5 pad 13: /Microcontroller/PA6 -> (no net)
- J5 pad 15: /Microcontroller/PA7 -> (no net)
- J5 pad 16: /Microcontroller/PB12 -> (no net)
- J5 pad 17: /Microcontroller/PB6 -> (no net)
- J5 pad 18: Net-(J5-Pad18) -> (no net)
- J5 pad 19: /Microcontroller/PC7 -> (no net)
- J5 pad 22: /Microcontroller/PB2 -> (no net)
- J5 pad 24: /Microcontroller/PB1 -> (no net)
- J5 pad 25: /Microcontroller/PB10 -> (no net)
- J5 pad 26: /Microcontroller/PB15 -> (no net)
- J5 pad 27: /Microcontroller/PB4 -> (no net)
- J5 pad 28: /Microcontroller/PB14 -> (no net)
- J5 pad 29: /Microcontroller/PB5 -> (no net)
- J5 pad 3: /Microcontroller/PB8 -> (no net)
- J5 pad 30: /Microcontroller/PB13 -> (no net)
- J5 pad 31: /Microcontroller/PB3 -> (no net)
- J5 pad 34: /Microcontroller/PC4 -> (no net)
- J5 pad 35: /Microcontroller/PA2 -> (no net)
- J5 pad 36: Net-(J5-Pad36) -> (no net)
- J5 pad 37: /Microcontroller/PA3 -> (no net)
- J5 pad 38: Net-(J5-Pad38) -> (no net)
- J5 pad 5: /Microcontroller/PB9 -> (no net)
- J5 pad 7: /Microcontroller/AVDD -> (no net)
- J5 pad 8: /Microcontroller/U5V -> (no net)
- U1 pad 1: Net-(U1-Pad1) -> (no net)
- U1 pad 3: Net-(U1-Pad3) -> (no net)
- U1 pad 5: Net-(U1-Pad5) -> (no net)
- U1 pad 8: Net-(U1-Pad8) -> (no net)
- U2 pad 1: Net-(U2-Pad1) -> (no net)
- U2 pad 5: /Input/BIAS -> (no net)
- U2 pad 6: (no net) -> /Input/BIAS
- U2 pad 8: Net-(U2-Pad8) -> (no net)
- U3 pad 4: Net-(U3-Pad4) -> (no net)
- U5 pad 4: Net-(U5-Pad4) -> (no net)
- U7 pad 7: Net-(U7-Pad7) -> (no net)
- U8 pad 7: Net-(U8-Pad7) -> (no net)
Routing:
- net /ADC/DB1: track 57.7 -> 61.4 mm
- net /ADC/DB2: track 56.2 -> 60.0 mm
- net /ADC/DB0: track 59.2 -> 63.0 mm
- net /ADC/DB3: track 49.8 -> 53.5 mm
- net /ADC/DB4: track 48.3 -> 52.1 mm
- net /ADC/DB5: track 37.1 -> 40.9 mm
- net /ADC/DB6: track 35.7 -> 39.4 mm
- net /Input/BIAS: track 107.4 -> 104.4 mm, vias 7 -> 6
- net /ADC/~SYNC: track 63.2 -> 66.0 mm
- net /ADC/DB14: track 35.9 -> 38.7 mm
- net /ADC/DB15: track 40.7 -> 43.5 mm
- net /ADC/~DRDY: track 58.7 -> 61.4 mm
- net /ADC/~CS: track 44.4 -> 47.1 mm
- net /ADC/~RESET: track 58.5 -> 61.2 mm
- net /ADC/~RD: track 46.3 -> 49.0 mm
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- added copper zone on F.Cu, net +2V5
Other:
- board text added: "DB0"
- board text added: "DB1"
- board text added: "DB10"
- board text added: "DB11"
- board text added: "DB12"
- board text added: "DB13"
- board text added: "DB14"
- board text added: "DB15"
- board text added: "DB2"
- board text added: "DB3"
- board text added: "DB4"
- board text added: "DB5"
- board text added: "DB6"
- board text added: "DB7"
- board text added: "DB8"
- board text added: "DB9"
- board text added: "Rev A 2018/04/12"
- board text added: "~CS"
- board text added: "~DRDY"
- board text added: "~RD"
- board text added: "~RESET"
- board text added: "~SYNC"
