File: ecad/input.sch (KiCad schematic (older format))
At the start: 0 parts

Commit message: Mostly complete schematic, about to tape out the PCB.
Parts:
- added C13, C14: 2.2u, Capacitors_SMD:C_0805_HandSoldering, symbol C
- added C15, C16: 47p, Capacitors_SMD:C_0603_HandSoldering, symbol C
- added C17, C18: 220p, Capacitors_SMD:C_0603_HandSoldering, symbol C
- added C19, C22, C25, C28, C39, C7: 0.1u, Capacitors_SMD:C_0603_HandSoldering, symbol C
- added C20, C21, C26, C27: 100p, Capacitors_SMD:C_0603_HandSoldering, symbol C
- added C23, C24: 1.5n, Capacitors_SMD:C_0603_HandSoldering, symbol C
- added C37, C38: 20p, Capacitors_SMD:C_0603_HandSoldering, symbol C
- added J2: XLR3, Pin_Headers:Pin_Header_Straight_1x03_Pitch2.54mm, symbol XLR3
- added R10: 1M, Resistors_SMD:R_0603_HandSoldering, symbol R
- added R11: 1MR, Resistors_SMD:R_0603_HandSoldering, symbol R
- added R12, R13, R14, R15: 349, Resistors_SMD:R_0603_HandSoldering, symbol R
- added R16, R17, R20, R21: 1k05, Resistors_SMD:R_0603_HandSoldering, symbol R
- added R18, R19: 698, Resistors_SMD:R_0603_HandSoldering, symbol R
- added R22, R23: 367, Resistors_SMD:R_0603_HandSoldering, symbol R
- added R24, R25: 332, Resistors_SMD:R_0603_HandSoldering, symbol R
- added R26, R27: 220, Resistors_SMD:R_0603_HandSoldering, symbol R
- added U6: OPA1612, Housings_SOIC:SOIC-8_3.9x4.9mm_Pitch1.27mm, symbol OPA1612
- added U7, U8: OPA1632, Housings_SOIC:SOIC-8_3.9x4.9mm_Pitch1.27mm, symbol OPA1632
Connections:
- new net: C13.2, J2.2
- new net: C14.2, J2.3
- new net: C13.1, R10.1, U6.3 (+)
- new net: C14.1, R11.2, U6.5 (+)
- new net: C21.2, R19.1, U7.1 (Vin-)
- new net: C21.1, R21.1, R22.2, U7.4 (Vout+)
- new net: C20.1, R20.1, R23.2, U7.5 (Vout-)
- new net: C20.2, R18.1, U7.8 (Vin+)
- new net: C15.1, R14.1, R17.2, U6.1
- new net: C15.2, R12.2, R14.2, U6.2 (-)
- new net: C16.2, R13.2, R15.2, U6.6 (-)
- new net: C16.1, R15.1, R16.2, U6.7
- new net: C17.1, C37.1, R17.1, R18.2, R20.2
- new net: C18.1, C38.1, R16.1, R19.2, R21.2
- new net: C27.2, R25.1, U8.1 (Vin-)
- new net: C26.2, R24.1, U8.8 (Vin+)
- new net: C23.1, R23.1, R24.2, R26.2
- new net: C24.1, R22.1, R25.2, R27.2
- new net +12: C22.1, C28.1, C39.1, U6.8, U7.3 (V+), U8.3 (V+)
- new net BIAS: C19.1, C25.1, C7.1, R10.2, R11.1, R12.1, R13.1, U7.2 (CM), U8.2 (CM)
- new net GND: C17.2, C18.2, C19.2, C22.2, C23.2, C24.2, C25.2, C28.2, C37.2, C38.2, C39.2, C7.2, J2.1, U6.4, U7.6 (V-), U8.6 (V-)
- new net PreOutN: C26.1, R26.1, U8.5 (Vout-)
- new net PreOutP: C27.1, R27.1, U8.4 (Vout+)
- no-connect marks 0 -> 2

Commit message: First complete pass of PCB with preamp, ADC, and nucleo dev board connections.
Connections:
- net PreOutN: now also C27.1, R27.1, U8.4 (Vout+); no longer C26.1, R26.1, U8.5 (Vout-)
- net PreOutP: now also C26.1, R26.1, U8.5 (Vout-); no longer C27.1, R27.1, U8.4 (Vout+)
Changed lines of the file:
@@
 $Descr A4 11693 8268
 encoding utf-8
-Sheet 3 5
+Sheet 2 5
 Title ""
 Date ""
@@
 P 5450 3750
 F 0 "U7" H 5450 3750 60  0000 C CNN
-F 1 "OPA1632" H 5850 4000 60  0000 C CNN
+F 1 "OPA1632" H 5300 3500 60  0000 C CNN
 F 2 "Housings_SOIC:SOIC-8_3.9x4.9mm_Pitch1.27mm" H 5450 3750 60  0001 C CNN
 F 3 "" H 5450 3750 60  0001 C CNN
@@
 P 7400 3750
 F 0 "U8" H 7400 3750 60  0000 C CNN
-F 1 "OPA1632" H 7800 4000 60  0000 C CNN
+F 1 "OPA1632" H 7250 3500 60  0000 C CNN
 F 2 "Housings_SOIC:SOIC-8_3.9x4.9mm_Pitch1.27mm" H 7400 3750 60  0001 C CNN
 F 3 "" H 7400 3750 60  0001 C CNN
@@
 $EndComp
 Text HLabel 8100 3850 2    60   Output ~ 0
+PreOutN
+Text HLabel 8100 3650 2    60   Output ~ 0
 PreOutP
-Text HLabel 8100 3650 2    60   Output ~ 0
-PreOutN
 $Comp
 L OPA1612 U6

Commit message: Rev A of board as ordered from Osh Park.
Parts:
- R11: value 1MR -> 1M
Other:
- note added: "4th Order LPF at 2 MHz"
- note added: "72.3mHz"
- note added: "9.7MHz\n"
- note added: "Enable is internally \ntied high with \n50k resistor."
- note added: "R12, R13, C15, C16 not populated\nR14 and R15 zero ohm."
- note added: "Since bias is 1/2 \nsupply, it is not \nstrictly necessary \nhere, but it may \nbe lower noise \nto feed in the \nlow impedance \nsource so we \nwill go with it."
Changed lines of the file:
@@
 P 2950 3950
 F 0 "R11" V 3030 3950 50  0000 C CNN
-F 1 "1MR" V 2950 3950 50  0000 C CNN
+F 1 "1M" V 2950 3950 50  0000 C CNN
 F 2 "Resistors_SMD:R_0603_HandSoldering" V 2880 3950 50  0001 C CNN
 F 3 "" H 2950 3950 50  0001 C CNN
@@
 Wire Wire Line
 	5600 1900 5600 2000
-Wire Wire Line
-	5150 1950 5300 1950
-Connection ~ 5300 1950
 Wire Wire Line
 	5300 2350 5300 2300
@@
 Text HLabel 3450 5050 3    60   Input ~ 0
 BIAS
-Text HLabel 5150 1950 0    60   Input ~ 0
-BIAS
 Text HLabel 7100 1950 0    60   Input ~ 0
 BIAS
@@
 Connection ~ 2650 3550
 Connection ~ 2950 3550
+Text Notes 2650 2950 0    60   ~ 0
+72.3mHz
+Text Notes 3850 3650 0    60   ~ 0
+9.7MHz\n
+Text Notes 5850 2700 0    60   ~ 0
+4th Order LPF at 2 MHz
+Text Notes 3250 2800 0    60   ~ 0
+R12, R13, C15, C16 not populated\nR14 and R15 zero ohm.
+Connection ~ 5300 1950
+Text HLabel 5150 1950 0    60   Input ~ 0
+BIAS
+Wire Wire Line
+	5150 1950 5300 1950
+Text Notes 6250 1600 0    60   ~ 0
+Since bias is 1/2 \nsupply, it is not \nstrictly necessary \nhere, but it may \nbe lower noise \nto feed in the \nlow impedance \nsource so we \nwill go with it.
+Text Notes 4450 1150 0    60   ~ 0
+Enable is internally \ntied high with \n50k resistor.
 $EndSCHEMATC

Commit message: Source track binary file.
Parts:
- R22, R23: value 367 -> 365
Changed lines of the file:
@@
 P 6350 3150
 F 0 "R23" V 6430 3150 50  0000 C CNN
-F 1 "367" V 6350 3150 50  0000 C CNN
+F 1 "365" V 6350 3150 50  0000 C CNN
 F 2 "Resistors_SMD:R_0603_HandSoldering" V 6280 3150 50  0001 C CNN
 F 3 "" H 6350 3150 50  0001 C CNN
@@
 P 6300 4250
 F 0 "R22" V 6380 4250 50  0000 C CNN
-F 1 "367" V 6300 4250 50  0000 C CNN
+F 1 "365" V 6300 4250 50  0000 C CNN
 F 2 "Resistors_SMD:R_0603_HandSoldering" V 6230 4250 50  0001 C CNN
 F 3 "" H 6300 4250 50  0001 C CNN
