File: ecad/input.sch (KiCad schematic (older format))
At the start: 40 parts, among them J2 XLR3, U6 OPA1612, U7 OPA1632, U8 OPA1632

Commit message: Slight changes to simulation and ecad with new changes before rollback to old changes.
Connections:
- wire segments 121 -> 117
Other:
- moved on the sheet: C13, C14, C15, C16, C17, C18, C19, C20, C21, C22, C23, C24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
